File: Hardware/Basic/HopeToPass-BASIC.sch (EAGLE design)
At the start: 52 parts, among them SW1 SWITCH.MOM, SW2 SWITCH.MOM, SW5 SWITCH.MOM, U2 NRF52832_MODULE_MDBT42, U4 PCF8523

Commit message: Complete eagle 001 and started programming
Parts:
- removed SW5: SWITCH.MOM, LinnesLab-Switches:SWITCH.MOM
Connections:
- removed net N$21: SW1.3, SW1.4
- removed net N$22: SW1.1
- removed net VBATT: U4.VBAT
- new net SW1: SW1.1, SW2.1
- net GND: now also SW1.3, SW1.4, SW2.3, SW2.4
Other:
- note added: "Buttons"
- note added: "Cortex Debugger"
- note added: "Power Management"
- note added: "RTC"
- note added: "Real-Time Clock"
- note added: "SD card"
- note added: "nRFS2832 M"
- note removed: "Back-up battery if desired"
- moved on the sheet: C10, C11, C12, C14, C2, C20, C21, C5, C6, C7, C8, C9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

Commit message: 10/16 updates
Parts:
- removed C2: 1u, LinnesLab-Passives:CAPACITOR0603
- removed SD2: (no value), LinnesLab-Connectors:MICROSD
- removed U4: PCF8523, LinnesLab-Clocks:PCF8523
- removed USB2: USB.MICRO-BIGGERPADS, LinnesLab-Connectors:USB.MICRO-BIGGERPADS
- removed XTAL3: 32.7680kHz, LinnesLab-Clocks:CRYSTALECS-.327-12.5-12-C-TR
- added C3: 1u, LinnesLab-Passives:CAPACITOR0603
- added J1: FTDI_DEVICESMD, LinnesLab-Connectors:FTDI_DEVICESMD
- added J3: (no value), LinnesLab-Connectors:CONN_07-1.27MM
- added U5: PCF8523, LinnesLab-Clocks:PCF8523
- added XTAL4: 32.7680kHz, LinnesLab-Clocks:CRYSTALECS-.327-12.5-12-C-TR
- C13, C15, C17, C18, C19: device LinnesLab-Passives:CAPACITOR0402 -> LinnesLab-Passives:CAPACITOR0603
Connections:
- net CHRG.STAT renamed D27/CHRG.STAT
- removed net BATT: R13.1, R14.2
- removed net CD1: SD2.CARD_DETECT
- removed net CD2: SD2.CARD_DETECT1
- removed net CS.OLED: U3./CS
- removed net DC.OLED: U3.DC/I2C_SA0
- removed net N$19: U4.OSCO, XTAL3.1
- removed net N$20: U4.OSCI, XTAL3.2
- removed net RESET.OLED: U3./RES
- removed net RXD: U2.P0.08
- removed net SD.CS: SD2.CS
- removed net SW1: SW1.1, SW2.1
- removed net TXD: U2.P0.06
- removed net USB+: USB2.D+
- removed net USB-: USB2.D-
- new net A4/PPG: J3.7, U2.P0.28/AIN4
- new net A5/TIA: J3.6, U2.P0.29/AIN5
- new net A7/BATT: R13.1, R14.2, U2.P0.31/AIN7
- new net D11/SW1: SW1.1, U2.P0.11
- new net D15/SW2: SW2.1, U2.P0.15
- new net D16/CS.OLED: U2.P0.16, U3./CS
- new net D27/CHRG.STATUS: U2.P0.27
- new net D3/RESET.OLED: U2.P0.03/AIN1, U3./RES
- new net D30/LED.CTRL: J3.5, U2.P0.30/AIN6
- new net D4/DC.OLED: U2.P0.04/AIN2, U3.DC/I2C_SA0
- new net D5/CD1: U2.P0.05/AIN3
- new net D7/SD.CS: U2.P0.07
- new net N$21: U5.OSCO, XTAL4.1
- new net N$22: U5.OSCI, XTAL4.2
- new net RXD.NRF: J1.TXO, U2.P0.08
- new net TXD.NRF: J1.RXI, U2.P0.06
- new net VBATT: U5.VBAT
- net 3.3V: now also C3.1, J3.4, U5.VDD; no longer C2.1, SD2.VDD, U4.VDD
- net DTR: now also J1.DTR
- net GND: now also C3.2, J1.CTS, J1.GND, J3.3, U5.VSS; no longer C2.2, SD2.GND, SD2.GND1, SD2.VSS, U4.VSS, USB2.GND
- net MISO: no longer SD2.DATA_OUT
- net MOSI: no longer SD2.DATA_IN
- net SCK: no longer SD2.SCLK
- net SCL: now also J3.2, U5.SCL; no longer U4.SCL
- net SDA: now also J3.1, U5.SDA; no longer U4.SDA
- net V_USB: now also J1.VCC; no longer USB2.V+
Other:
- note added: "Back-up battery if desired"
- note added: "Headers connecting top and bottom board"
- note removed: "Connect MISO, MOSI, and SCK to appropriate pins on microcontroller. Those are SPI pins and are generally prespecified. You have more flexibility with the SD.CS pin."
- note removed: "SD card"
- moved on the sheet: R8, R9, SW4

Commit message: Completed Routing the board
Parts:
- removed C10, C11: 300p, LinnesLab-Passives:CAPACITOR0603
- removed R15: 100k, LinnesLab-Passives:RESISTOR0603
Connections:
- removed net D27/CHRG.STAT: CHRG2.STAT, R12.1
- removed net P0.09/NFC1: C11.1, U2.P0.09
- removed net P0.10/NFC2: C10.1, U2.P0.10
- net 3.3V: no longer R15.2
- net D27/CHRG.STATUS: now also CHRG2.STAT, R12.1
- net GND: no longer C10.2, C11.2, R15.1, SW1.4, SW2.4
Changed lines of the file:
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@@
 <part name="GND15" library="LinnesLab-Symbols" deviceset="GND" device=""/>
 <part name="GND16" library="LinnesLab-Symbols" deviceset="GND" device=""/>
-<part name="GND17" library="LinnesLab-Symbols" deviceset="GND" device=""/>
-<part name="GND18" library="LinnesLab-Symbols" deviceset="GND" device=""/>
 <part name="GND19" library="LinnesLab-Symbols" deviceset="GND" device=""/>
 <part name="GND20" library="LinnesLab-Symbols" deviceset="GND" device=""/>
@@
 <part name="C8" library="LinnesLab-Passives" deviceset="CAPACITOR" device="0603" package3d_urn="urn:adsk.eagle:package:15661989/2"/>
 <part name="C9" library="LinnesLab-Passives" deviceset="CAPACITOR" device="0603" package3d_urn="urn:adsk.eagle:package:15661989/2"/>
-<part name="C10" library="LinnesLab-Passives" deviceset="CAPACITOR" device="0603" package3d_urn="urn:adsk.eagle:package:15661989/2" value="300p"/>
-<part name="C11" library="LinnesLab-Passives" deviceset="CAPACITOR" device="0603" package3d_urn="urn:adsk.eagle:package:15661989/2" value="300p"/>
 <part name="C12" library="LinnesLab-Passives" deviceset="CAPACITOR" device="0805" package3d_urn="urn:adsk.eagle:package:15662010/2" value="10u"/>
 <part name="L2" library="LinnesLab-Passives" deviceset="INDUCTOR" device="0603" override_package3d_urn="urn:adsk.eagle:package:18592195/2" override_package_urn="urn:adsk.eagle:footprint:18592196/1" value="10u"/>
@@
 <part name="SUPPLY16" library="LinnesLab-Symbols" deviceset="VLIPO" device=""/>
 <part name="GND43" library="LinnesLab-Symbols" deviceset="GND" device=""/>
-<part name="R15" library="LinnesLab-Passives" deviceset="RESISTOR" device="0603" package3d_urn="urn:adsk.eagle:package:15661944/2" value="100k"/>
-<part name="GND44" library="LinnesLab-Symbols" deviceset="GND" device=""/>
 <part name="SUPPLY17" library="LinnesLab-Symbols" deviceset="VIN" device=""/>
 <part name="SW1" library="LinnesLab-Switches" deviceset="SWITCH.MOM" device=""/>
@@
 <attribute name="VALUE" x="55.88" y="101.346" size="1.778" layer="96" align="top-center"/>
 </instance>
-<instance part="GND17" gate="G$1" x="58.42" y="71.12" smashed="yes">
-<attribute name="VALUE" x="58.42" y="70.866" size="1.778" layer="96" align="top-center"/>
-</instance>
-<instance part="GND18" gate="G$1" x="45.72" y="71.12" smashed="yes">
-<attribute name="VALUE" x="45.72" y="70.866" size="1.778" layer="96" align="top-center"/>
-</instance>
 <instance part="GND19" gate="G$1" x="35.56" y="71.12" smashed="yes">
 <attribute name="VALUE" x="35.56" y="70.866" size="1.778" layer="96" align="top-center"/>
@@
 <attribute name="VALUE" x="37.084" y="76.581" size="1.778" layer="96"/>
 </instance>
-<instance part="C10" gate="G$1" x="58.42" y="78.74" smashed="yes">
-<attribute name="NAME" x="59.944" y="81.661" size="1.778" layer="95"/>
-<attribute name="VALUE" x="59.944" y="76.581" size="1.778" layer="96"/>
-</instance>
-<instance part="C11" gate="G$1" x="45.72" y="78.74" smashed="yes">
-<attribute name="NAME" x="47.244" y="81.661" size="1.778" layer="95"/>
-<attribute name="VALUE" x="47.244" y="76.581" size="1.778" layer="96"/>
-</instance>
 <instance part="C12" gate="G$1" x="15.24" y="114.3" smashed="yes" rot="R180">
 <attribute name="NAME" x="13.716" y="111.379" size="1.778" layer="95" rot="R180"/>
@@
 <instance part="GND43" gate="G$1" x="190.5" y="-30.48" smashed="yes">
 <attribute name="VALUE" x="190.5" y="-30.734" size="1.778" layer="96" align="top-center"/>
-</instance>
-<instance part="R15" gate="G$1" x="203.2" y="5.08" smashed="yes" rot="R90">
-<attribute name="NAME" x="201.7014" y="1.27" size="1.778" layer="95" rot="R90"/>
-<attribute name="VALUE" x="206.502" y="1.27" size="1.778" layer="96" rot="R90"/>
-</instance>
-<instance part="GND44" gate="G$1" x="203.2" y="-5.08" smashed="yes">
-<attribute name="VALUE" x="203.2" y="-5.334" size="1.778" layer="96" align="top-center"/>
 </instance>
 <instance part="SUPPLY17" gate="G$1" x="144.78" y="15.24" smashed="yes">
@@
 <pinref part="GND20" gate="G$1" pin="GND"/>
 <pinref part="C8" gate="G$1" pin="1"/>
-</segment>
-<segment>
-<pinref part="C11" gate="G$1" pin="2"/>
-<pinref part="GND18" gate="G$1" pin="GND"/>
-<wire x1="45.72" y1="73.66" x2="45.72" y2="76.2" width="0.1524" layer="91"/>
-</segment>
-<segment>
-<pinref part="C10" gate="G$1" pin="2"/>
-<pinref part="GND17" gate="G$1" pin="GND"/>
-<wire x1="58.42" y1="73.66" x2="58.42" y2="76.2" width="0.1524" layer="91"/>
 </segment>
 <segment>
@@
 </segment>
 <segment>
-<pinref part="R15" gate="G$1" pin="1"/>
-<pinref part="GND44" gate="G$1" pin="GND"/>
-<wire x1="203.2" y1="-2.54" x2="203.2" y2="0" width="0.1524" layer="91"/>
-</segment>
-<segment>
 <pinref part="SW1" gate="G$1" pin="3"/>
 <wire x1="289.56" y1="55.88" x2="294.64" y2="55.88" width="0.1524" layer="91"/>
-<wire x1="294.64" y1="55.88" x2="294.64" y2="53.34" width="0.1524" layer="91"/>
-<pinref part="SW1" gate="G$1" pin="4"/>
-<wire x1="294.64" y1="53.34" x2="294.64" y2="45.72" width="0.1524" layer="91"/>
-<wire x1="289.56" y1="53.34" x2="294.64" y2="53.34" width="0.1524" layer="91"/>
-<junction x="294.64" y="53.34"/>
+<wire x1="294.64" y1="55.88" x2="294.64" y2="45.72" width="0.1524" layer="91"/>
 <pinref part="GND1" gate="G$1" pin="GND"/>
 </segment>
@@
 <pinref part="SW2" gate="G$1" pin="3"/>
 <wire x1="325.12" y1="55.88" x2="330.2" y2="55.88" width="0.1524" layer="91"/>
-<wire x1="330.2" y1="55.88" x2="330.2" y2="53.34" width="0.1524" layer="91"/>
-<pinref part="SW2" gate="G$1" pin="4"/>
-<wire x1="330.2" y1="53.34" x2="330.2" y2="45.72" width="0.1524" layer="91"/>
-<wire x1="325.12" y1="53.34" x2="330.2" y2="53.34" width="0.1524" layer="91"/>
-<junction x="330.2" y="53.34"/>
+<wire x1="330.2" y1="55.88" x2="330.2" y2="45.72" width="0.1524" layer="91"/>
 <pinref part="GND2" gate="G$1" pin="GND"/>
 </segment>
@@
 <wire x1="193.04" y1="15.24" x2="193.04" y2="12.7" width="0.1524" layer="91"/>
 <junction x="193.04" y="12.7"/>
-<wire x1="193.04" y1="12.7" x2="203.2" y2="12.7" width="0.1524" layer="91"/>
-<pinref part="R15" gate="G$1" pin="2"/>
-<wire x1="203.2" y1="12.7" x2="203.2" y2="10.16" width="0.1524" layer="91"/>
 </segment>
 <segment>
@@
 </segment>
 </net>
-<net name="P0.09/NFC1" class="0">
-<segment>
-<wire x1="50.8" y1="106.68" x2="50.8" y2="86.36" width="0.1524" layer="91"/>
-<wire x1="45.72" y1="86.36" x2="50.8" y2="86.36" width="0.1524" layer="91"/>
-<wire x1="45.72" y1="86.36" x2="45.72" y2="83.82" width="0.1524" layer="91"/>
-<pinref part="C11" gate="G$1" pin="1"/>
-<pinref part="U2" gate="G$1" pin="P0.09"/>
-<label x="50.8" y="88.9" size="1.27" layer="95" rot="R180" xref="yes"/>
-</segment>
-</net>
 <net name="SCK" class="0">
 <segment>
@@
 <wire x1="104.14" y1="-12.7" x2="109.22" y2="-12.7" width="0.1524" layer="91"/>
 <label x="109.22" y="-12.7" size="1.778" layer="95" xref="yes"/>
-</segment>
-</net>
-<net name="P0.10/NFC2" class="0">
-<segment>
-<wire x1="53.34" y1="106.68" x2="53.34" y2="86.36" width="0.1524" layer="91"/>
-<wire x1="53.34" y1="86.36" x2="58.42" y2="86.36" width="0.1524" layer="91"/>
-<wire x1="58.42" y1="86.36" x2="58.42" y2="83.82" width="0.1524" layer="91"/>
-<pinref part="C10" gate="G$1" pin="1"/>
-<pinref part="U2" gate="G$1" pin="P0.10"/>
-<label x="53.34" y="88.9" size="1.27" layer="95" xref="yes"/>
 </segment>
 </net>
@@
 <pinref part="J1" gate="G$1" pin="VCC"/>
 <wire x1="104.14" y1="-20.32" x2="127" y2="-20.32" width="0.1524" layer="91"/>
-</segment>
-</net>
-<net name="D27/CHRG.STAT" class="0">
-<segment>
-<pinref part="R12" gate="G$1" pin="1"/>
-<wire x1="160.02" y1="-33.02" x2="160.02" y2="-38.1" width="0.1524" layer="91"/>
-<wire x1="160.02" y1="-38.1" x2="165.1" y2="-38.1" width="0.1524" layer="91"/>
-<wire x1="165.1" y1="-38.1" x2="165.1" y2="-25.4" width="0.1524" layer="91"/>
-<pinref part="CHRG2" gate="G$1" pin="STAT"/>
-<wire x1="165.1" y1="-25.4" x2="167.64" y2="-25.4" width="0.1524" layer="91"/>
-<label x="165.1" y="-38.1" size="1.27" layer="95" xref="yes"/>
 </segment>
 </net>
@@
 <label x="15.24" y="139.7" size="1.27" layer="95" rot="R180" xref="yes"/>
 </segment>
-</net>
+<segment>
+<pinref part="R12" gate="G$1" pin="1"/>
+<wire x1="160.02" y1="-33.02" x2="160.02" y2="-38.1" width="0.1524" layer="91"/>
+<wire x1="160.02" y1="-38.1" x2="165.1" y2="-38.1" width="0.1524" layer="91"/>
+<wire x1="165.1" y1="-38.1" x2="165.1" y2="-25.4" width="0.1524" layer="91"/>
+<pinref part="CHRG2" gate="G$1" pin="STAT"/>
+<wire x1="165.1" y1="-25.4" x2="167.64" y2="-25.4" width="0.1524" layer="91"/>
+<label x="165.1" y="-38.1" size="1.27" layer="95" xref="yes"/>
+</segment>
+</net>

Commit message: orlando renumbered components
Parts:
- removed C17, C18, C19: 2.2uF, LinnesLab-Passives:CAPACITOR0603
- removed C20, C21: 4.7u, LinnesLab-Passives:CAPACITOR0603
- removed D4: (no value), LinnesLab-DiscreteSemi:SCHOTTKY-USC
- removed R12, R13, R14: 100k, LinnesLab-Passives:RESISTOR0603
- removed U5: PCF8523, LinnesLab-Clocks:PCF8523
- removed XTAL4: 32.7680kHz, LinnesLab-Clocks:CRYSTALECS-.327-12.5-12-C-TR
- added C1: 1u, LinnesLab-Passives:CAPACITOR0603
- added C10: 10uF, LinnesLab-Passives:CAPACITOR0603
- added C11: 2.2uF, LinnesLab-Passives:CAPACITOR0603
- added C2: 10u, LinnesLab-Passives:CAPACITOR0805
- added C4: 22p, LinnesLab-Passives:CAPACITOR0603
- added D3: (no value), LinnesLab-DiscreteSemi:SCHOTTKY-USC
- added R1, R2: 1k, LinnesLab-Passives:RESISTOR0603
- added R10: 10k, LinnesLab-Passives:RESISTOR0603
- added U1: NRF52832_MODULE_MDBT42, LinnesLab-Microcontrollers:NRF52832_MODULE_MDBT42
- added XTAL1: 32.768kHz, LinnesLab-Clocks:CRYSTALECS-.327-12.5-12-C-TR
- C12: value 10u -> 2.2uF; device LinnesLab-Passives:CAPACITOR0805 -> LinnesLab-Passives:CAPACITOR0603
- C14: value 100n -> 2.2uF
- C16: value 10uF -> 1u
- C3: value 1u -> 22p
- C5: value 1u -> 4.7u
- C8: value (none) -> 4.7u
- C9: value (none) -> 100n
- J1: value FTDI_DEVICESMD -> (none); device LinnesLab-Connectors:FTDI_DEVICESMD -> LinnesLab-Connectors:CONN_07-1.27MM
- J2: value (none) -> FTDI_DEVICESMD; device LinnesLab-Connectors:CONN_02 -> LinnesLab-Connectors:FTDI_DEVICESMD
- J3: device LinnesLab-Connectors:CONN_07-1.27MM -> LinnesLab-Connectors:CONN_02
- R11: value (none) -> 10k
- R3: value 1k -> 100k
- R4: value 1k -> 4.7k
- R6: value 10k -> 100k
- R7: value 390k -> 100k
- R9: value 10k -> 390k
- SW1, SW2: value SWITCH.MOM -> (none); device LinnesLab-Switches:SWITCH.MOM -> LinnesLab-Switches:SPST-PTS830GG140-COPY.1-3
- SW3, SW4: value (none) -> SWITCH.MOM; device LinnesLab-Switches:SPST-PTS830GG140-COPY.1-3 -> LinnesLab-Switches:SWITCH.MOM
- U2: value NRF52832_MODULE_MDBT42 -> PCF8523; device LinnesLab-Microcontrollers:NRF52832_MODULE_MDBT42 -> LinnesLab-Clocks:PCF8523; DIGIKEY (none) -> 568-5306-1-ND; I2C_ADDRESS (none) -> 0x68h; MFN (none) -> PCF8523T/1,118; MFN_MANUFACTURER (none) -> NXP USA Inc.
- XTAL2: value 32.768kHz -> 32.7680kHz; FREQ (none) -> 32.7680KHZ
- renumbered CHRG2 to CHRG1, CORTEX1 to DEBUG1, D5 to D2, L2 to L1, LDO2 to LDO1, LED3 to LED1, LED4 to LED2
Connections:
- net 3.3V: now also C14.2, C15.2, C16.1, C2.2, C7.1, D3.C, J1.4, R10.2, R11.2, U1.VDD; no longer C12.2, C17.2, C19.2, C3.1, C6.1, D1.C, J3.4, R8.2, R9.2, U5.VDD
- net A4/PPG: now also J1.7, U1.P0.28/AIN4; no longer J3.7, U2.P0.28/AIN4
- net A5/TIA: now also J1.6, U1.P0.29/AIN5; no longer J3.6, U2.P0.29/AIN5
- net A7/BATT: now also R6.1, R7.2, U1.P0.31/AIN7; no longer R13.1, R14.2, U2.P0.31/AIN7
- net D11/SW1: now also SW3.1, U1.P0.11; no longer SW1.1, U2.P0.11
- net D15/SW2: now also SW4.1, U1.P0.15; no longer SW2.1, U2.P0.15
- net D16/CS.OLED: now also U1.P0.16; no longer U2.P0.16
- net D27/CHRG.STATUS: now also R3.1, U1.P0.27; no longer R12.1, U2.P0.27
- net D3/RESET.OLED: now also U1.P0.03/AIN1; no longer U2.P0.03/AIN1
- net D30/LED.CTRL: now also J1.5, U1.P0.30/AIN6; no longer J3.5, U2.P0.30/AIN6
- net D4/DC.OLED: now also U1.P0.04/AIN2; no longer U2.P0.04/AIN2
- net D5/CD1: now also U1.P0.05/AIN3; no longer U2.P0.05/AIN3
- net D7/SD.CS: now also U1.P0.07; no longer U2.P0.07
- net DFU: now also SW1.B, U1.P0.20; no longer SW3.B, U2.P0.20
- net DTR: now also C9.1, J2.DTR; no longer C14.1, J1.DTR
- net FRST: now also U1.P0.22; no longer U2.P0.22
- net GND: now also C1.2, C10.1, C14.1, C15.1, C16.2, C2.1, C3.1, C4.2, C6.1, C8.2, J1.3, J2.CTS, J2.GND, J3.1, R4.1, R7.1, R8.1, R9.2, SW1.A, SW2.B, SW3.3, SW4.3, U1.GND@1, U1.GND@2, U1.GND@3, U1.GND@4, U2.VSS; no longer C16.1, C17.1, C18.1, C19.1, C20.2, C21.1, C3.2, C6.2, C8.1, C9.2, J1.CTS, J1.GND, J2.1, J3.3, R11.1, R14.1, R6.1, R7.2, SW1.3, SW2.3, SW3.A, SW4.B, U2.GND@1, U2.GND@2, U2.GND@3, U2.GND@4, U5.VSS
- net LED1: now also R1.2, U1.P0.17; no longer R3.2, U2.P0.17
- net LED2: now also R2.2, U1.P0.19; no longer R4.2, U2.P0.19
- net MISO: now also U1.P0.14; no longer U2.P0.14
- net MOSI: now also U1.P0.13; no longer U2.P0.13
- net N$1: now also R8.2; no longer R6.2
- net N$10: now also R2.1; no longer R4.1
- net N$11: now also U1.DCC; no longer U2.DCC
- net N$12: now also C1.1, U1.DEC4; no longer C7.1, U2.DEC4
- net N$13: now also C10.2; no longer C16.2
- net N$15: now also C12.2; no longer C18.2
- net N$17: now also R4.2; no longer R11.2
- net N$2: now also R9.1; no longer R7.1
- net N$21: now also U2.OSCO, XTAL2.1; no longer U5.OSCO, XTAL4.1
- net N$22: now also U2.OSCI, XTAL2.2; no longer U5.OSCI, XTAL4.2
- net N$4: now also C3.2, U1.P0.00/XL1, XTAL1.1; no longer C8.2, U2.P0.00/XL1, XTAL2.1
- net N$6: now also C4.1, U1.P0.01/XL2, XTAL1.2; no longer C9.1, U2.P0.01/XL2, XTAL2.2
- net N$7: now also C11.2; no longer C15.2
- net N$8: now also C11.1; no longer C15.1
- net N$9: now also R1.1; no longer R3.1
- net RESET: now also C9.2, D3.A, SW2.A, U1.P0.21/RESET; no longer C14.2, D1.A, SW4.A, U2.P0.21/RESET
- net RXD.NRF: now also J2.TXO, U1.P0.08; no longer J1.TXO, U2.P0.08
- net SCK: now also U1.P0.12; no longer U2.P0.12
- net SCL: now also J1.2, R10.1, U1.P0.26, U2.SCL; no longer J3.2, R8.1, U2.P0.26, U5.SCL
- net SDA: now also J1.1, R11.1, U1.P0.25, U2.SDA; no longer J3.1, R9.1, U2.P0.25, U5.SDA
- net SWCLK: now also U1.SWDCLK; no longer U2.SWDCLK
- net SWDIO: now also U1.SWDIO; no longer U2.SWDIO
- net SWO: now also U1.P0.18/SWO; no longer U2.P0.18/SWO
- net TXD.NRF: now also J2.RXI, U1.P0.06; no longer J1.RXI, U2.P0.06
- net VBATT: now also U2.VBAT; no longer U5.VBAT
- net VIN: now also C6.2, D1.C, R3.2; no longer C21.2, D4.C, R12.2
- net VLIPO: now also C8.1, D1.A, J3.2, R6.2; no longer C20.1, D4.A, J2.2, R13.2
- net V_USB: now also J2.VCC; no longer J1.VCC
Other:
- moved on the sheet: C12, C14, C15, C16, C3, C5, C6, C7, C8, C9, D1, R11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
